File: Sweep half-swept/half-swept.kicad_pcb (KiCad board)
At the start: 2 copper layers, 109 x 86.6 mm, 28 parts, among them J2 AudioJack4dpb, SW1 SW_Push, SW10 SW_Push, SW11 SW_Push, SW12 SW_Push, SW13 SW_Push, SW14 SW_Push, SW15 SW_Push, SW16 SW_Push, SW17 SW_Push, SW2 SW_Push, SW3 SW_Push, SW4 SW_Push, SW5 SW_Push, SW6 SW_Push, SW7 SW_Push, SW8 SW_Push, SW9 SW_Push, U1 ProMicro-kbd

Commit message: Remove assembly instructions from silkscreen
Other:
- board text removed: "1) Place Pro-Micro with components facing DOWN"
- board text removed: "2) Close JUMPER PADS on the OPPOSITE SIDE"
Changed lines of the file:
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@@
     (effects (font (size 0.6 0.6) (thickness 0.15)) (justify mirror))
-  )
-  (gr_text "2) Close JUMPER PADS\non the OPPOSITE SIDE" (at 121.7168 53.7464 90) (layer "B.SilkS")
-    (effects (font (size 1 1) (thickness 0.15) italic) (justify left mirror))
   )
   (gr_text "GND" (at 116.40097 51.6128) (layer "B.SilkS")
     (effects (font (size 0.6 0.6) (thickness 0.12)) (justify left mirror))
   )
-  (gr_text "1) Place Pro-Micro with\ncomponents facing DOWN" (at 115.9764 53.7464 90) (layer "B.SilkS")
-    (effects (font (size 1 1) (thickness 0.15) italic) (justify left mirror))
-  )
   (gr_text "B+" (at 124.587 45.974) (layer "B.SilkS")
     (effects (font (size 0.6 0.6) (thickness 0.15)) (justify mirror))
-  )
-  (gr_text "1) Place Pro-Micro with\ncomponents facing DOWN" (at 115.9764 72.4408 90) (layer "F.SilkS")
-    (effects (font (size 1 1) (thickness 0.15) italic) (justify left))
   )
   (gr_text "GND" (at 121.3612 51.6128) (layer "F.SilkS")
     (effects (font (size 0.6 0.6) (thickness 0.12)) (justify left))
   )
-  (gr_text "2) Close JUMPER PADS\non the OPPOSITE SIDE" (at 121.8692 72.4408 90) (layer "F.SilkS")
-    (effects (font (size 1 1) (thickness 0.15) italic) (justify left))
-  )
   (gr_text "RAW" (at 121.3612 49.0728) (layer "F.SilkS")

Commit message: Remove TRRS
Parts:
- removed J2: AudioJack4dpb, Kailh:TRRS-PJ-DPB2
Routing:
- net vcc: track 47.9 -> 0.00 mm, vias 4 -> 0
- net Switch18: track 34.2 -> 0.00 mm
Changed lines of the file:
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@@
     )
   )
-  (footprint "Kailh:TRRS-PJ-DPB2" (layer "F.Cu")
-    (at 123.698 82.75 -90)
-    (attr through_hole)
-    (fp_text reference "J2" (at -0.85 4.95 180) (layer "F.Fab") hide
-      (effects (font (size 1 1) (thickness 0.15)))
-    )
-    (fp_text value "AudioJack4dpb" (at 0 14 90) (layer "F.Fab") hide
-      (effects (font (size 1 1) (thickness 0.15)))
-    )
-    (fp_text user "TRRS" (at -0.073 4.826 180) (layer "B.SilkS") hide
-      (effects (font (size 1 1) (thickness 0.15)) (justify mirror))
-    )
-    (fp_text user "Ring2" (at 0 3.25 90) (layer "F.Fab") hide
-      (effects (font (size 0.7 0.7) (thickness 0.1)))
-    )
-    (fp_text user "Ring1" (at 0 6.25 90) (layer "F.Fab") hide
-      (effects (font (size 0.7 0.7) (thickness 0.1)))
-    )
-    (fp_text user "Tip" (at 0 10 90) (layer "F.Fab") hide
-      (effects (font (size 0.7 0.7) (thickness 0.1)))
-    )
-    (fp_text user "Sleeve" (at 0.25 11.4 90) (layer "F.Fab") hide
-      (effects (font (size 0.7 0.7) (thickness 0.1)))
-    )
-    (pad "R1" thru_hole oval (at -2.33 6.22 90) (size 1.6 2) (drill oval 0.9 1.3) (layers *.Cu *.Mask)
-      (net 3 "Switch18"))
-    (pad "R1" thru_hole oval (at 2.3 6.2 270) (size 1.6 2) (drill oval 0.9 1.3) (layers *.Cu *.Mask)
-      (net 3 "Switch18"))
-    (pad "R2" thru_hole oval (at 2.3 3.2 270) (size 1.6 2) (drill oval 0.9 1.3) (layers *.Cu *.Mask)
-      (net 2 "vcc"))
-    (pad "R2" thru_hole oval (at -2.33 3.22 90) (size 1.6 2) (drill oval 0.9 1.3) (layers *.Cu *.Mask)
-      (net 2 "vcc"))
-    (pad "S" thru_hole oval (at -2.3 11.3 270) (size 1.6 2) (drill oval 0.9 1.3) (layers *.Cu *.Mask)
-      (net 1 "gnd"))
-    (pad "S" thru_hole oval (at 2.27 11.32 90) (size 1.6 2) (drill oval 0.9 1.3) (layers *.Cu *.Mask)
-      (net 1 "gnd"))
-    (pad "T" thru_hole oval (at -2.33 10.22 90) (size 1.6 2) (drill oval 0.9 1.3) (layers *.Cu *.Mask)
-      (net 1 "gnd"))
-    (pad "T" thru_hole oval (at 2.3 10.2 270) (size 1.6 2) (drill oval 0.9 1.3) (layers *.Cu *.Mask)
-      (net 1 "gnd"))
-    (model "/Users/danny/syncproj/kicad-libs/footprints/Keebio-Parts.pretty/3dmodels/PJ-320A.step"
-      (offset (xyz 0 0 0))
-      (scale (xyz 1 1 1))
-      (rotate (xyz -90 0 180))
-    )
-  )
   (footprint "Sweep half-swept:SW_PG1350_rev_DPB" (layer "F.Cu")
     (at 27.08 46.08)
@@
   (arc (start 110.3946 49.8794) (mid 110.690465 50.077091) (end 111.039462 50.146511) (width 0.25) (layer "B.Cu") (net 1))
   (arc (start 110.127489 49.234537) (mid 110.196908 49.583534) (end 110.3946 49.8794) (width 0.25) (layer "B.Cu") (net 1))
-  (segment (start 120.498 80.454142) (end 120.498 85.05) (width 0.25) (layer "F.Cu") (net 2))
-  (segment (start 108.5596 58.212751) (end 108.5596 61.4172) (width 0.25) (layer "F.Cu") (net 2))
-  (segment (start 106.045 70.0024) (end 106.0196 70.0024) (width 0.25) (layer "F.Cu") (net 2))
-  (segment (start 108.5596 67.5132) (end 106.08836 69.984439) (width 0.25) (layer "F.Cu") (net 2))
-  (segment (start 120.488 80.43) (end 120.478 80.42) (width 0.25) (layer "F.Cu") (net 2))
-  (segment (start 109.347 56.3118) (end 110.1344 55.5244) (width 0.25) (layer "F.Cu") (net 2))
-  (via (at 106.0196 70.0024) (size 0.8) (drill 0.4) (layers "F.Cu" "B.Cu") (net 2))
-  (via (at 110.1344 55.5244) (size 0.8) (drill 0.4) (layers "F.Cu" "B.Cu") (net 2))
-  (via (at 108.5596 67.5132) (size 0.8) (drill 0.4) (layers "F.Cu" "B.Cu") (net 2))
-  (via (at 108.5596 61.4172) (size 0.8) (drill 0.4) (layers "F.Cu" "B.Cu") (net 2))
-  (arc (start 120.488 80.43) (mid 120.495401 80.441076) (end 120.498 80.454142) (width 0.25) (layer "F.Cu") (net 2))
-  (arc (start 109.347 56.3118) (mid 108.764238 57.183963) (end 108.5596 58.212751) (width 0.25) (layer "F.Cu") (net 2))
-  (arc (start 106.08836 69.984439) (mid 106.068466 69.997732) (end 106.045 70.0024) (width 0.25) (layer "F.Cu") (net 2))
-  (segment (start 108.5596 67.5132) (end 108.5596 61.4172) (width 0.25) (layer "B.Cu") (net 2))
-  (segment (start 113.912363 81.8388) (end 118.055956 81.8388) (width 0.25) (layer "B.Cu") (net 2))
-  (segment (start 110.146197 55.517489) (end 112.126339 55.517489) (width 0.25) (layer "B.Cu") (net 2))
-  (segment (start 113.483744 56.079744) (end 114.046 56.642) (width 0.25) (layer "B.Cu") (net 2))
-  (segment (start 119.7686 81.1294) (end 120.478 80.42) (width 0.25) (layer "B.Cu") (net 2))
-  (segment (start 106.0196 73.946036) (end 106.0196 70.0024) (width 0.25) (layer "B.Cu") (net 2))
-  (segment (start 110.1344 55.5244) (end 110.137855 55.520944) (width 0.25) (layer "B.Cu") (net 2))
-  (segment (start 110.064607 80.245007) (end 107.613392 77.793792) (width 0.25) (layer "B.Cu") (net 2))
-  (arc (start 110.064607 80.245007) (mid 111.829972 81.424586) (end 113.912363 81.8388) (width 0.25) (layer "B.Cu") (net 2))
-  (arc (start 110.146197 55.517489) (mid 110.141682 55.518386) (end 110.137855 55.520944) (width 0.25) (layer "B.Cu") (net 2))
-  (arc (start 106.0196 73.946036) (mid 106.433813 76.028426) (end 107.613392 77.793792) (width 0.25) (layer "B.Cu") (net 2))
-  (arc (start 119.7686 81.1294) (mid 118.982832 81.654432) (end 118.055956 81.8388) (width 0.25) (layer "B.Cu") (net 2))
-  (arc (start 113.483744 56.079744) (mid 112.860961 55.663614) (end 112.126339 55.517489) (width 0.25) (layer "B.Cu") (net 2))
-  (segment (start 118.472255 51.924255) (end 118.11 51.562) (width 0.25) (layer "F.Cu") (net 3))
-  (segment (start 118.834511 52.798817) (end 118.834511 78.10429) (width 0.25) (layer "F.Cu") (net 3))
-  (segment (start 118.156255 79.741744) (end 117.488 80.41) (width 0.25) (layer "F.Cu") (net 3))
-  (segment (start 117.498 80.454142) (end 117.498 85.05) (width 0.25) (layer "F.Cu") (net 3))
-  (arc (start 117.488 80.41) (mid 117.483857 80.42) (end 117.488 80.43) (width 0.25) (layer "F.Cu") (net 3))
-  (arc (start 117.488 80.43) (mid 117.495401 80.441076) (end 117.498 80.454142) (width 0.25) (layer "F.Cu") (net 3))
-  (arc (start 118.834511 78.10429) (mid 118.658238 78.990474) (end 118.156255 79.741744) (width 0.25) (layer "F.Cu") (net 3))
-  (arc (start 118.472255 51.924255) (mid 118.740363 52.325507) (end 118.834511 52.798817) (width 0.25) (layer "F.Cu") (net 3))
   (segment (start 87.3252 22.2504) (end 86.4852 22.2504) (width 0.25) (layer "F.Cu") (net 4))
   (via (at 87.3252 22.2504) (size 0.8) (drill 0.4) (layers "F.Cu" "B.Cu") (net 4))

Commit message: Move Rust logo, make it larger
Parts:
- removed the G*** at (118.2, 83.6) (x2)
- removed the G*** at (64.0, 82.0)
- added G***: LOGO, Sweep half-swept:rust_larger, B.Cu at (63.2, 79.4)
